File: micarray/micarray.kicad_sch (KiCad schematic)
At the start: 37 parts, among them IC1 74LCX125MTCX, J1 Previous, J2 Next, J3 MCHStreamer J3

Commit message: Save before dev-fork
Parts:
- C11: value 20p -> 150p
Changed lines of the file:
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@@
 			)
 		)
-		(property "Value" "20p"
+		(property "Value" "150p"
 			(at 223.5199 50.8 0)
 			(effects
