File: micarry_8ch_camera/micarry_8ch_camera.kicad_sch (KiCad schematic)
At the start: 68 parts, among them IC1 74LCX125MTCX, IC2 74LCX125MTCX, J1 MCHStreamer J3

Commit message: 8ch progress, new mics for 16ch
Parts:
- J1: footprint Connector_PinHeader_2.54mm:PinHeader_2x06_P2.54mm_Vertical -> Connector_PinHeader_2.00mm:PinHeader_2x06_P2.00mm_Vertical
Connections:
- net PDM_CLK0: now also R18.1; no longer R19.1
- net PDM_CLK1: now also R19.1; no longer R18.1
- net PDM_CLK4: now also R23.1; no longer R24.1
- net PDM_CLK5: now also R24.1; no longer R23.1
Changed lines of the file:
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@@
 	(global_label "PDM_CLK1"
 		(shape input)
+		(at 39.37 252.73 180)
+		(fields_autoplaced yes)
+		(effects
+			(font
+				(size 1.27 1.27)
+			)
+			(justify right)
+		)
+		(property "Intersheetrefs" "${INTERSHEET_REFS}"
+			(at 26.6482 252.73 0)
+			(effects
+				(font
+					(size 1.27 1.27)
+				)
+				(justify right)
+				(hide yes)
+			)
+		)
+	)
+	(global_label "PDM_CLK1"
+		(shape input)
 		(at 34.29 93.98 180)
 		(fields_autoplaced yes)
@@
 		)
 	)
-	(global_label "PDM_CLK4"
+	(global_label "PDM_CLK5"
 		(shape input)
-		(at 186.69 69.85 180)
+		(at 181.61 252.73 180)
 		(fields_autoplaced yes)
 		(effects
@@
 		)
 		(property "Intersheetrefs" "${INTERSHEET_REFS}"
-			(at 173.9682 69.85 0)
+			(at 168.8882 252.73 0)
 			(effects
 				(font
@@
 		)
 	)
-	(global_label "PDM_DATA0"
+	(global_label "PDM_CLK4"
 		(shape input)
-		(at 102.87 91.44 0)
+		(at 186.69 69.85 180)
 		(fields_autoplaced yes)
 		(effects
@@
 				(size 1.27 1.27)
 			)
-			(justify left)
+			(justify right)
 		)
 		(property "Intersheetrefs" "${INTERSHEET_REFS}"
-			(at 116.4385 91.44 0)
+			(at 173.9682 69.85 0)
 			(effects
 				(font
 					(size 1.27 1.27)
 				)
-				(justify left)
+				(justify right)
 				(hide yes)
 			)
 		)
 	)
-	(global_label "PDM_DATA3"
+	(global_label "PDM_CLK0"
 		(shape input)
-		(at 255.27 140.97 0)
+		(at 39.37 245.11 180)
 		(fields_autoplaced yes)
 		(effects
@@
 				(size 1.27 1.27)
 			)
-			(justify left)
+			(justify right)
 		)
 		(property "Intersheetrefs" "${INTERSHEET_REFS}"
-			(at 268.8385 140.97 0)
+			(at 26.6482 245.11 0)
 			(effects
 				(font
 					(size 1.27 1.27)
 				)
-				(justify left)
+				(justify right)
 				(hide yes)
 			)
 		)
 	)
-	(global_label "PDM_DATA1"
+	(global_label "PDM_DATA0"
 		(shape input)
-		(at 102.87 140.97 0)
+		(at 102.87 91.44 0)
 		(fields_autoplaced yes)
 		(effects
@@
 		)
 		(property "Intersheetrefs" "${INTERSHEET_REFS}"
-			(at 116.4385 140.97 0)
+			(at 116.4385 91.44 0)
 			(effects
 				(font
@@
 		)
 	)
-	(global_label "PDM_CLK0"
+	(global_label "PDM_CLK4"
 		(shape input)
-		(at 39.37 252.73 180)
+		(at 181.61 245.11 180)
 		(fields_autoplaced yes)
 		(effects
@@
 		)
 		(property "Intersheetrefs" "${INTERSHEET_REFS}"
-			(at 26.6482 252.73 0)
+			(at 168.8882 245.11 0)
 			(effects
 				(font
@@
 		)
 	)
-	(global_label "PDM_CLK5"
+	(global_label "PDM_DATA3"
 		(shape input)
-		(at 181.61 245.11 180)
+		(at 255.27 140.97 0)
 		(fields_autoplaced yes)
 		(effects
@@
 				(size 1.27 1.27)
 			)
-			(justify right)
+			(justify left)
 		)
 		(property "Intersheetrefs" "${INTERSHEET_REFS}"
-			(at 168.8882 245.11 0)
+			(at 268.8385 140.97 0)
 			(effects
 				(font
 					(size 1.27 1.27)
 				)
-				(justify right)
+				(justify left)
 				(hide yes)
 			)
 		)
 	)
-	(global_label "PDM_CLK5"
+	(global_label "PDM_DATA1"
 		(shape input)
-		(at 186.69 93.98 180)
+		(at 102.87 140.97 0)
 		(fields_autoplaced yes)
 		(effects
@@
 				(size 1.27 1.27)
 			)
-			(justify right)
+			(justify left)
 		)
 		(property "Intersheetrefs" "${INTERSHEET_REFS}"
-			(at 173.9682 93.98 0)
+			(at 116.4385 140.97 0)
 			(effects
 				(font
 					(size 1.27 1.27)
 				)
-				(justify right)
+				(justify left)
 				(hide yes)
 			)
 		)
 	)
-	(global_label "PDM_CLK4"
+	(global_label "PDM_CLK5"
 		(shape input)
-		(at 181.61 252.73 180)
+		(at 186.69 93.98 180)
 		(fields_autoplaced yes)
 		(effects
@@
 		)
 		(property "Intersheetrefs" "${INTERSHEET_REFS}"
-			(at 168.8882 252.73 0)
+			(at 173.9682 93.98 0)
 			(effects
 				(font
@@
 		)
 	)
-	(global_label "PDM_CLK1"
-		(shape input)
-		(at 39.37 245.11 180)
-		(fields_autoplaced yes)
-		(effects
-			(font
-				(size 1.27 1.27)
-			)
-			(justify right)
-		)
-		(property "Intersheetrefs" "${INTERSHEET_REFS}"
-			(at 26.6482 245.11 0)
-			(effects
-				(font
-					(size 1.27 1.27)
-				)
-				(justify right)
-				(hide yes)
-			)
-		)
-	)
 	(global_label "PDM_CLK3"
 		(shape input)
@@
 			)
 		)
-		(property "Footprint" "Connector_PinHeader_2.54mm:PinHeader_2x06_P2.54mm_Vertical"
+		(property "Footprint" "Connector_PinHeader_2.00mm:PinHeader_2x06_P2.00mm_Vertical"
 			(at 31.75 35.56 0)
 			(effects

Commit message: Save before dev-fork
Parts:
- removed MK1, MK2, MK3, MK4, MK5, MK6, MK7, MK8: SPH1668LM4H-1, Sensor_Audio:Knowles_LGA-5_3.5x2.65mm, symbol SPH1668LM4H-1:SPH1668LM4H-1
- added MK1, MK2, MK3, MK4, MK5, MK6, MK7, MK8: ~, ul_IM73D122V01XTMA1:PG-LLGA-5-2_INF, symbol ProLib_pcs_2024-08-11:IM73D122V01XTMA1
Connections:
- net +3V3: no longer C21.1
- net GND: now also MK1.4 (LR), MK1.5 (GND), MK2.5 (GND), MK3.4 (LR), MK3.5 (GND), MK4.5 (GND), MK5.4 (LR), MK5.5 (GND), MK6.5 (GND), MK7.4 (LR), MK7.5 (GND), MK8.5 (GND)
- net PDM_CLK-IN: now also C21.1
- net PDM_CLK0: now also R1.2; no longer R1.1
- net PDM_CLK2: now also R5.2; no longer R5.1
- net PDM_CLK3: now also R7.2; no longer R7.1
- net PDM_CLK4: now also R9.2; no longer R9.1
- net PDM_CLK6: now also R13.2; no longer R13.1
- net PDM_CLK7: now also R15.2; no longer R15.1
- net at R10.1: now also MK5.1 (DATA)
- net at R16.1: now also MK8.1 (DATA)
- net at C10.2, C9.2, L5.1: now also MK5.2 (VDD)
- net at C5.2, C6.2, L3.1: now also MK3.2 (VDD)
- net at C11.2, C12.2, L6.1: now also MK6.2 (VDD), MK6.4 (LR)
- net at C7.2, C8.2, L4.1: now also MK4.2 (VDD), MK4.4 (LR)
- net at C15.2, C16.2, L8.1: now also MK8.2 (VDD), MK8.4 (LR)
- net at R6.1: now also MK3.1 (DATA)
- net at C13.2, C14.2, L7.1: now also MK7.2 (VDD)
- net at R11.2: now also MK6.3 (CLOCK)
- net at R14.1: now also MK7.1 (DATA)
- net at C1.2, C2.2, L1.1: now also MK1.2 (VDD)
- net at R3.2: now also MK2.3 (CLOCK)
- net at C3.2, C4.2, L2.1: now also MK2.2 (VDD), MK2.4 (LR)
- net at R8.1: now also MK4.1 (DATA)
- net at R2.1: now also MK1.1 (DATA)
- net at R4.1: now also MK2.1 (DATA)
- net at R12.1: now also MK6.1 (DATA)
- new net: MK7.3 (CLOCK), R13.1
- new net: MK3.3 (CLOCK), R5.1
- new net: MK1.3 (CLOCK), R1.1
- new net: MK4.3 (CLOCK), R7.1
- new net: MK8.3 (CLOCK), R15.1
- new net: MK5.3 (CLOCK), R9.1
Other:
- moved on the sheet: C1, C2, C3, C4, C5, C6, C7, C8, L1, L2, L3, L4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
